File: hardware/KiCad/shaper_amplifier.kicad_sch (KiCad schematic)
At the start: 27 parts, among them Q1 2SK932, U3 OPA818IDRG, U4 OPA1632DGN, U5 AD8099ARD

Commit message: More schemataic tidying. Added a csa_core_simulation.kicad_pro to simulate CSA core. Tidied csa_core to make it simulatable, but needs work - OP analysis doesn't converge at the moment. (Need to fiddle with op-amp compensation??)
Parts:
- removed C15, C19, C8: 0.1uF, Capacitor_SMD:C_0805_2012Metric, symbol Device:C_Small
- removed C17, C7: 10uF, Capacitor_SMD:C_0805_2012Metric, symbol Device:C
- removed C25: 0.5pF CQ0805BRNPO0BNR50, Capacitor_SMD:C_0805_2012Metric_Pad1.18x1.45mm_HandSolder, symbol Device:C_Small
- removed Q1: 2SK932, Package_TO_SOT_SMD:SOT-23, symbol 2SK932:2SK932
- removed R11: 2M, Resistor_SMD:R_0603_1608Metric_Pad0.98x0.95mm_HandSolder, symbol Device:R
- removed R13: 100M CRCW1206100MJPEAHR, Resistor_SMD:R_1206_3216Metric_Pad1.30x1.75mm_HandSolder, symbol Device:R
- removed TP1: TestPoint, TestPoint:TestPoint_Pad_2.0x2.0mm, symbol Connector:TestPoint
- removed U3: OPA818IDRG, Package_SON:WSON-8-1EP_3x3mm_P0.5mm_EP1.45x2.4mm, symbol Amplifier_Operational:OPA818xDRG
- removed U5: AD8099ARD, AD8099:RD_8_1_ADI, symbol AD8099:AD8099ARD
- added C18, C20, C24: 0.1uF, Capacitor_SMD:C_0805_2012Metric, symbol Device:C_Small
- added C19: 10uF, Capacitor_SMD:C_0805_2012Metric, symbol Device:C
- added TP3: TestPoint, TestPoint:TestPoint_Pad_2.0x2.0mm, symbol Connector:TestPoint
- C21: value 2.2p -> 10uF; footprint Resistor_SMD:R_0603_1608Metric_Pad0.98x0.95mm_HandSolder -> Capacitor_SMD:C_0805_2012Metric
- renumbered C11 to C22, C14 to C23, C13 to C25, C9 to C26, C10 to C27, C16 to C28, C18 to C29, R4 to R11, R6 to R12, R3 to R13, R9 to R14, R5 to R15, R7 to R16, U4 to U6
Connections:
- net +6V is gone; now on net V+: C26.1, C27.1, U6.3 (V+)
- net -6V is gone; now on net V-: C28.1, C29.1, U6.6 (V-)
- net GND: now also C21.2, C18.2, C19.2, C20.2, C24.1
- net V+: now also C18.1, C19.1
- net V-: now also C21.1, C20.1
- net Vocm: now also C24.2
- net Vin: now reaches R11.2
- net Vin: now also TP3.1
Other:
- note removed: "Equivalent noise charge (ENC)* ENC RMS 200 electrons 0.03 femtoCoul. Equivalent noise in silicon 1.7 keV (FWHM) Equivalent noise in CdZnTe 2.4 keV (FWHM)"
- note removed: "IP no load 250mA, upto 400mA OP 250uA adjust voltage 1 to 5V giving upto 2500V"
- note removed: "Optimal PS +/-6V"
- note removed: "Tdecay = 1.4pF x 100M = 140us Trise = 3ns for CR-110-R2.1"
