File: hardware/KiCad/csa_core_phase_margin_simulation/csa_core_phase_margin_simulation.kicad_sch (KiCad schematic)
At the start: 23 parts, among them Q1 MMDT3906, Q2 2SK932, U1 ${SIM.PARAMS}

Commit message: Generated artwork
Parts:
- removed Q1: MMDT3906, Package_TO_SOT_SMD:SOT-363_SC-70-6, symbol Transistor_BJT:MMDT3906
- added C10: 1uF, Capacitor_SMD:C_0805_2012Metric, symbol Device:C_Small
- added Q1: BFS20, Package_TO_SOT_SMD:SOT-23, symbol BFS20:BFS20
- added R7: 1.2k, Resistor_SMD:R_0603_1608Metric, symbol Device:R
- added R8: 1k, Resistor_SMD:R_0603_1608Metric, symbol Device:R
- R1: value 560 -> 1k
- R3: value 1k -> 2.2k
- R5: value 100 -> 10
- R6: value 100 -> 1000
- V1: value 6 -> 10
Connections:
- net GND: now also C10.1
- net V+: now also R7.1, R8.1
- net vfet: now also Q1.3 (C), R8.2; no longer Q2.2 (D)
- net mirror_base renamed vbase
- net vbase: now also C10.2, Q1.1 (B), R7.2
- new net ve: Q1.2 (E), Q2.2 (D)
Other:
- moved on the sheet: R1

Commit message: Produced gerbers
Parts:
- R3: value 2.2k -> 1.5k
Changed lines of the file:
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@@
 			)
 		)
-		(property "Value" "2.2k"
+		(property "Value" "1.5k"
 			(at 154.94 148.5899 0)
 			(effects
